File: Hardware/Schematics/KiCad/v1/v1.kicad_pcb (KiCad board)
At the start: 2 copper layers, 8 parts, among them SW1 SW_Push_Dual_x2, SW2 SW_Push_Dual_x2, U1 OLED_128x32, U2 GY-271_QMC5883L, U3 GY-61_ADXL335

Commit message: fixed adxl pinout
Connections:
- U3 pad 1: /GND -> /VCC
- U3 pad 5: /VCC -> /GND
Routing:
- net /VCC: track 203.2 -> 191.2 mm
- net /GND: track 216.5 -> 212.6 mm
