File: Hardware/Schematics/KiCad/v1/v1.sch (KiCad schematic (older format))
At the start: 8 parts, among them SW1 SW_Push_Dual_x2, SW2 SW_Push_Dual_x2, U1 OLED_128x32, U2 GY-271_QMC5883L, U3 GY-61_ADXL335

Commit message: fixed adxl pinout
Connections:
- net GND: now also U3.5 (GND); no longer U3.1 (VCC)
- net VCC: now also U3.1 (VCC); no longer U3.5 (GND)
Changed lines of the file:
@@
 	4500 4000 4500 4550
-Wire Wire Line
-	6800 3900 6800 3700
-Wire Wire Line
-	6800 3700 8050 3700
 Wire Wire Line
 	5650 2050 5650 2300
@@
 	6650 3050 8050 3050
 Connection ~ 8050 3050
-Wire Wire Line
-	8050 3050 8050 3700
 Text Label 7350 2050 0    50   ~ 0
 VCC
@@
 Text Label 7600 3050 0    50   ~ 0
 VCC
-Text Label 7700 3700 0    50   ~ 0
+Text Label 8050 3700 1    50   ~ 0
 VCC
 Text Label 6350 2900 0    50   ~ 0
@@
 Wire Wire Line
 	6050 4000 6800 4000
-Text Label 6300 3950 0    50   ~ 0
+Text Label 6550 3900 0    50   ~ 0
 GND
 Text Label 6600 3500 0    50   ~ 0
@@
 Connection ~ 5450 4550
 Wire Wire Line
-	6300 3300 6300 4300
-Wire Wire Line
-	6800 4300 6300 4300
-Connection ~ 6300 4300
-Wire Wire Line
-	6300 4300 6300 4550
+	6300 3300 6300 3900
 Text Label 6550 4000 0    50   ~ 0
 A2
@@
 	0    -1   -1   0
 $EndComp
+Wire Wire Line
+	6800 3900 6300 3900
+Connection ~ 6300 3900
+Wire Wire Line
+	6300 3900 6300 4550
+Wire Wire Line
+	6800 4300 6800 4450
+Wire Wire Line
+	6800 4450 8050 4450
+Wire Wire Line
+	8050 3050 8050 4450
 $EndSCHEMATC
